File: pcb_source/fourtyeighty.kicad_pcb (KiCad board)
At the start: 2 copper layers, 274.6 x 79.4 mm, 148 parts, among them J1 USB_C_Receptacle_USB2.0, SW1 RotaryEncoder_Switch, U1 XC6206PxxxMR, U2 SRV05-4, U3 W25Q128JVS, U4 RP2040TR7, Y1 Crystal_GND24_Small

Commit message: routed rows
Routing:
- net ROW2: track 0.00 -> 192.8 mm, vias 0 -> 6
- net ROW7: track 0.00 -> 138.9 mm
- net ROW5: track 0.00 -> 134.6 mm
- net ROW0: track 0.00 -> 129.7 mm
- net ROW1: track 0.00 -> 126.6 mm, vias 0 -> 4
- net ROW4: track 0.00 -> 126.6 mm
- net ROW6: track 0.00 -> 108.9 mm
- net ROW3: track 0.00 -> 92.4 mm
- net +5V: track 0.00 -> 14.6 mm
- net GND: track 58.6 -> 68.9 mm, vias 16 -> 20
- net +3V3: track 62.0 -> 64.0 mm

Commit message: A bit more routing
Routing:
- net +3V3: track 64.0 -> 156.0 mm
Changed lines of the file:
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@@
     (fp_arc (start 8.53125 -7.500001) (mid 8.677688 -7.853563) (end 9.03125 -8.000001)
       (stroke (width 0.05) (type solid)) (layer "Eco2.User"))
-    (fp_arc (start 9.03125 5.999999) (mid 8.677694 5.853541) (end 8.53125 5.499999)
+    (fp_arc (start 9.03125 5.999999) (mid 8.677729 5.853535) (end 8.53125 5.499999)
       (stroke (width 0.05) (type solid)) (layer "Eco2.User"))
-    (fp_arc (start 14.78125 -8.000001) (mid 15.134807 -7.853543) (end 15.28125 -7.500001)
+    (fp_arc (start 14.78125 -8.000001) (mid 15.134771 -7.853537) (end 15.28125 -7.500001)
       (stroke (width 0.05) (type solid)) (layer "Eco2.User"))
-    (fp_arc (start 15.280039 5.499999) (mid 15.133589 5.853531) (end 14.780039 5.999999)
+    (fp_arc (start 15.280039 5.499999) (mid 15.133581 5.853541) (end 14.780039 5.999999)
       (stroke (width 0.05) (type solid)) (layer "Eco2.User"))
     (pad "" np_thru_hole circle (at -11.90625 -8.255) (size 3.9878 3.9878) (drill 3.9878) (layers "*.Cu" "*.Mask"))
@@
     (fp_arc (start 1.749484 0.919721) (mid 1.638072 1.504036) (end 1.046711 1.5683)
       (stroke (width 0.1) (type solid)) (layer "Edge.Cuts"))
-    (fp_arc (start 1.749484 0.919721) (mid 1.712534 0.814067) (end 1.699999 0.702843)
+    (fp_arc (start 1.749484 0.919721) (mid 1.71254 0.814067) (end 1.699999 0.702843)
       (stroke (width 0.1) (type solid)) (layer "Edge.Cuts"))
     (fp_line (start -3.8 -1.999999) (end -3.8 2.000001)
@@
     (fp_arc (start 8.53125 -7.500001) (mid 8.677688 -7.853563) (end 9.03125 -8.000001)
       (stroke (width 0.05) (type solid)) (layer "Eco2.User"))
-    (fp_arc (start 9.03125 5.999999) (mid 8.677694 5.853541) (end 8.53125 5.499999)
+    (fp_arc (start 9.03125 5.999999) (mid 8.677729 5.853535) (end 8.53125 5.499999)
       (stroke (width 0.05) (type solid)) (layer "Eco2.User"))
-    (fp_arc (start 14.78125 -8.000001) (mid 15.134807 -7.853543) (end 15.28125 -7.500001)
+    (fp_arc (start 14.78125 -8.000001) (mid 15.134771 -7.853537) (end 15.28125 -7.500001)
       (stroke (width 0.05) (type solid)) (layer "Eco2.User"))
-    (fp_arc (start 15.280039 5.499999) (mid 15.133589 5.853531) (end 14.780039 5.999999)
+    (fp_arc (start 15.280039 5.499999) (mid 15.133581 5.853541) (end 14.780039 5.999999)
       (stroke (width 0.05) (type solid)) (layer "Eco2.User"))
     (pad "" np_thru_hole circle (at -11.90625 -8.255) (size 3.9878 3.9878) (drill 3.9878) (layers "*.Cu" "*.Mask"))
@@
   (segment (start 138.70625 83.521875) (end 138.70625 83.121875) (width 0.2) (layer "B.Cu") (net 3))
   (segment (start 135.46875 83.521875) (end 135.90625 83.521875) (width 0.2) (layer "B.Cu") (net 3))
+  (segment (start 41.58875 65.88125) (end 121.279359 65.88125) (width 0.25) (layer "B.Cu") (net 3))
   (segment (start 141.30625 83.921875) (end 141.30625 84.321875) (width 0.2) (layer "B.Cu") (net 3))
   (segment (start 138.70625 88.921875) (end 138.70625 89.559375) (width 0.2) (layer "B.Cu") (net 3))
@@
   (segment (start 136.50625 87.521875) (end 136.50625 88.121875) (width 0.2) (layer "B.Cu") (net 3))
   (segment (start 139.10625 83.721875) (end 140.90625 83.721875) (width 0.2) (layer "B.Cu") (net 3))
+  (segment (start 123.195641 66.675) (end 131.886268 66.675) (width 0.25) (layer "B.Cu") (net 3))
   (segment (start 134.14375 80.521875) (end 134.14375 80.251875) (width 0.2) (layer "B.Cu") (net 3))
   (segment (start 138.30625 82.684375) (end 138.70625 82.684375) (width 0.2) (layer "B.Cu") (net 3))
@@
   (arc (start 138.30625 83.321875) (mid 138.189093 83.604718) (end 137.90625 83.721875) (width 0.2) (layer "B.Cu") (net 3))
   (arc (start 140.90625 83.721875) (mid 141.189093 83.839032) (end 141.30625 84.121875) (width 0.2) (layer "B.Cu") (net 3))
+  (arc (start 40.795 65.0875) (mid 41.027484 65.648766) (end 41.58875 65.88125) (width 0.25) (layer "B.Cu") (net 3))
   (arc (start 141.70625 87.121875) (mid 141.423407 87.004718) (end 141.30625 86.721875) (width 0.2) (layer "B.Cu") (net 3))
   (arc (start 136.50625 84.121875) (mid 136.623407 83.839032) (end 136.90625 83.721875) (width 0.2) (layer "B.Cu") (net 3))
+  (arc (start 121.279359 65.88125) (mid 121.797901 65.984394) (end 122.2375 66.278125) (width 0.25) (layer "B.Cu") (net 3))
   (arc (start 138.70625 88.921875) (mid 138.823407 88.639032) (end 139.10625 88.521875) (width 0.2) (layer "B.Cu") (net 3))
+  (arc (start 122.2375 66.278125) (mid 122.677098 66.571856) (end 123.195641 66.675) (width 0.25) (layer "B.Cu") (net 3))
   (arc (start 138.70625 83.321875) (mid 138.823407 83.604718) (end 139.10625 83.721875) (width 0.2) (layer "B.Cu") (net 3))
   (arc (start 136.10625 83.521875) (mid 136.389093 83.639032) (end 136.50625 83.921875) (width 0.2) (layer "B.Cu") (net 3))
   (arc (start 141.70625 83.521875) (mid 141.423407 83.639032) (end 141.30625 83.921875) (width 0.2) (layer "B.Cu") (net 3))
   (arc (start 136.10625 87.121875) (mid 136.389093 87.004718) (end 136.50625 86.721875) (width 0.2) (layer "B.Cu") (net 3))
+  (arc (start 131.886268 66.675) (mid 132.034073 66.6456) (end 132.159375 66.561875) (width 0.25) (layer "B.Cu") (net 3))
   (arc (start 138.30625 83.521875) (mid 138.364829 83.663296) (end 138.50625 83.721875) (width 0.2) (layer "B.Cu") (net 3))
   (arc (start 134.78625 75.841875) (mid 134.938554 75.474179) (end 135.30625 75.321875) (width 0.2) (layer "B.Cu") (net 3))

Commit message: almost done with columns
Parts:
- turned D1 to 0 degrees
- turned D2 to 0 degrees
- turned D27 to 0 degrees
- turned D28 to 0 degrees
Connections:
- MX1 pad 1: COL0 -> Net-(D1-A)
- MX1 pad 2: Net-(D1-A) -> COL0
- MX2 pad 1: COL1 -> Net-(D2-A)
- MX2 pad 2: Net-(D2-A) -> COL1
- MX27 pad 1: COL5 -> Net-(D27-A)
- MX27 pad 2: Net-(D27-A) -> COL5
- MX28 pad 1: COL6 -> Net-(D28-A)
- MX28 pad 2: Net-(D28-A) -> COL6
- U4 pad 12: unconnected-(U4-GPIO9-Pad12) -> RGB
- U4 pad 13: unconnected-(U4-GPIO10-Pad13) -> ROW7
- U4 pad 2: unconnected-(U4-GPIO0-Pad2) -> COL6
- U4 pad 3: unconnected-(U4-GPIO1-Pad3) -> ROW0
- U4 pad 30: unconnected-(U4-GPIO19-Pad30) -> ROW3
- U4 pad 31: unconnected-(U4-GPIO20-Pad31) -> COL5
- U4 pad 35: unconnected-(U4-GPIO23-Pad35) -> ROW2
- U4 pad 36: unconnected-(U4-GPIO24-Pad36) -> ROW1
- U4 pad 37: unconnected-(U4-GPIO25-Pad37) -> COL4
- U4 pad 38: unconnected-(U4-GPIO26/ADC0-Pad38) -> COL3
- U4 pad 39: unconnected-(U4-GPIO27/ADC1-Pad39) -> COL2
- U4 pad 4: unconnected-(U4-GPIO2-Pad4) -> ROW4
- U4 pad 40: unconnected-(U4-GPIO28/ADC2-Pad40) -> COL1
- U4 pad 41: unconnected-(U4-GPIO29/ADC3-Pad41) -> COL0
- U4 pad 5: unconnected-(U4-GPIO3-Pad5) -> ROW5
- U4 pad 6: unconnected-(U4-GPIO4-Pad6) -> ROW6
- U4 pad 7: unconnected-(U4-GPIO5-Pad7) -> ENCB
- U4 pad 8: unconnected-(U4-GPIO6-Pad8) -> ENCA
Routing:
- net COL0: track 0.00 -> 232.7 mm, vias 0 -> 1
- net COL1: track 0.00 -> 205.6 mm, vias 0 -> 1
- net COL2: track 0.00 -> 194.2 mm, vias 0 -> 1
- net COL3: track 0.00 -> 175.1 mm, vias 0 -> 1
- net COL4: track 0.00 -> 164.8 mm, vias 0 -> 1
- net COL6: track 0.00 -> 130.9 mm, vias 0 -> 1
- net COL5: track 0.00 -> 126.5 mm, vias 0 -> 1
- net ROW0: track 129.7 -> 189.0 mm, vias 0 -> 1
- net ROW4: track 126.6 -> 185.8 mm, vias 0 -> 1
- net ROW1: track 126.6 -> 170.6 mm, vias 4 -> 6
- net ROW3: track 92.4 -> 130.7 mm
- net ROW5: track 134.6 -> 169.8 mm, vias 0 -> 1
- net ROW7: track 138.9 -> 174.0 mm
- net +3V3: track 156.0 -> 182.3 mm, vias 2 -> 4
- net ROW2: track 192.8 -> 216.8 mm, vias 6 -> 7
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
Commit message: Just a few more connections
Connections:
- U4 pad 7: ENCB -> ENCA
- U4 pad 8: ENCA -> ENCB
Routing:
- net +5V: track 14.6 -> 322.2 mm, vias 0 -> 4
- net ENCB: track 6.16 -> 172.6 mm
- net ENCA: track 6.16 -> 171.9 mm
- net RGB: track 6.80 -> 166.3 mm
- net ROW6: track 115.0 -> 138.2 mm
- net ROW5: track 169.8 -> 179.4 mm, vias 1 -> 2
- net ROW0: track 189.0 -> 198.2 mm, vias 1 -> 2
- net ROW4: track 185.8 -> 193.2 mm, vias 1 -> 2
- net GND: track 88.6 -> 92.7 mm, vias 21 -> 23
- net ROW2: track 216.8 -> 216.2 mm
