File: pcb_source/fourtyeighty.kicad_sch (KiCad schematic)
At the start: 148 parts, among them J1 USB_C_Receptacle_USB2.0, SW1 RotaryEncoder_Switch, U1 XC6206PxxxMR, U2 SRV05-4, U3 W25Q128JVS, U4 RP2040TR7, Y1 Crystal_GND24_Small

Commit message: almost done with columns
Connections:
- net COL0: now also MX1.2 (ROW), U4.41 (GPIO29/ADC3); no longer MX1.1 (COL)
- net COL1: now also MX2.2 (ROW), U4.40 (GPIO28/ADC2); no longer MX2.1 (COL)
- net COL2: now also U4.39 (GPIO27/ADC1)
- net COL3: now also U4.38 (GPIO26/ADC0)
- net COL4: now also U4.37 (GPIO25)
- net COL5: now also MX27.2 (ROW), U4.31 (GPIO20); no longer MX27.1 (COL)
- net COL6: now also MX28.2 (ROW), U4.2 (GPIO0); no longer MX28.1 (COL)
- net ENCA: now also U4.8 (GPIO6)
- net ENCB: now also U4.7 (GPIO5)
- net RGB: now also U4.12 (GPIO9)
- net ROW0: now also U4.3 (GPIO1)
- net ROW1: now also U4.36 (GPIO24)
- net ROW2: now also U4.35 (GPIO23)
- net ROW3: now also U4.30 (GPIO19)
- net ROW4: now also U4.4 (GPIO2)
- net ROW5: now also U4.5 (GPIO3)
- net ROW6: now also U4.6 (GPIO4)
- net ROW7: now also U4.13 (GPIO10)
- net at D28.2 (A): now also MX28.1 (COL); no longer MX28.2 (ROW)
- net at D1.2 (A): now also MX1.1 (COL); no longer MX1.2 (ROW)
- net at D27.2 (A): now also MX27.1 (COL); no longer MX27.2 (ROW)
- net at D2.2 (A): now also MX2.1 (COL); no longer MX2.2 (ROW)
Other:
- moved on the sheet: MX1, MX2, MX27, MX28

Commit message: Just a few more connections
Connections:
- net ENCA: now also U4.7 (GPIO5); no longer U4.8 (GPIO6)
- net ENCB: now also U4.8 (GPIO6); no longer U4.7 (GPIO5)
Changed lines of the file:
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@@
     )
   )
-  (global_label "ENCB" (shape input) (at 29.21 151.13 180) (fields_autoplaced)
-    (effects (font (size 1.27 1.27)) (justify right))
-    (property "Intersheetrefs" "${INTERSHEET_REFS}" (at 21.2847 151.13 0)
+  (global_label "ENCB" (shape input) (at 29.21 153.67 180) (fields_autoplaced)
+    (effects (font (size 1.27 1.27)) (justify right))
+    (property "Intersheetrefs" "${INTERSHEET_REFS}" (at 21.2847 153.67 0)
       (effects (font (size 1.27 1.27)) (justify right) hide)
     )
@@
     )
   )
-  (global_label "ENCA" (shape input) (at 29.21 153.67 180) (fields_autoplaced)
-    (effects (font (size 1.27 1.27)) (justify right))
-    (property "Intersheetrefs" "${INTERSHEET_REFS}" (at 21.4661 153.67 0)
-      (effects (font (size 1.27 1.27)) (justify right) hide)
-    )
+  (global_label "ENCA" (shape input) (at 29.21 151.13 180) (fields_autoplaced)
+    (effects (font (size 1.27 1.27)) (justify right))
+    (property "Intersheetrefs" "${INTERSHEET_REFS}" (at 21.4661 151.13 0)
+      (effects (font (size 1.27 1.27)) (justify right) hide)
+    )
