File: LowProTest/LowProTest.kicad_pcb (KiCad board)
At the start: 2 copper layers, 38.1 x 57.2 mm, 7 parts, among them SW1 SW_Push_45deg, SW2 SW_Push_45deg, SW7 SW_Push_45deg, SW8 SW_Push_45deg

Commit message: lo-pro test production
Parts:
- removed SW7: SW_Push_45deg, PCM_marbastlib-mx:SW_MX_1u
- removed the SW8 at (177.8, 108.3)
- added REF**: STAB_MX_2u, marbastlib-mx:STAB_MX_2u, F.Cu at (187.3, 127.4)
- added SW2: SW_Push_45deg, kiserdesigns:KS-33-HS, B.Cu at (177.8, 98.8)
Other:
- outline, holes or cut-outs redrawn
- board text added: "5.2"
- board text added: "5.25"
