File: HS_KS-SLD_MX/HS_KS-SLD_MX.kicad_pcb (KiCad board)
At the start: 2 copper layers, 274.6 x 84.1 mm, 148 parts, among them J1 USB_C_Receptacle_USB2.0, SW1 RotaryEncoder_Switch, U1 XC6206PxxxMR, U2 SRV05-4, U3 W25Q128JVS, U4 RP2040TR7, Y1 Crystal_GND24_Small

Commit message: Routed, will DRC tomorrow
Parts:
- removed C11: 100n, Capacitor_SMD:C_0402_1005Metric
- J1: footprint Connector_USB:USB_C_Receptacle_HRO_TYPE-C-31-M-12 -> PCM_marbastlib-various:USB_C_Receptacle_HRO_TYPE-C-31-M-12
- MX1, MX10, MX11, MX12, MX15, MX16, MX17, MX18, MX19, MX2, MX20, MX21, MX22, MX23, MX24, MX25, MX26, MX29, MX3, MX30, MX31, MX32, MX33, MX34, MX35, MX36, MX37, MX38, MX39, MX4, MX40, MX41, MX42, MX43, MX44, MX45, MX46, MX47, MX48, MX49, MX5, MX50, MX51, MX52, MX53, MX6, MX7, MX8, MX9: footprint kiserdesigns:HS-KS-33-MX -> kiserdesigns:HS-KS-33_Soldered-MX
- moved C1 102.7 mm to (143.3, 47.6)
- moved C2 102.7 mm to (143.3, 53.2)
- moved U1 102.7 mm to (143.3, 50.4)
- moved R1 98.0 mm to (137.3, 38.9)
- moved J1 97.7 mm to (138.9, 32.5)
- moved R2 97.2 mm to (140.5, 38.9)
- moved F1 94.1 mm to (138.9, 48.0), turned to 0 degrees
- moved U2 90.9 mm to (138.9, 51.2), turned to 180 degrees
- moved D14 31.3 mm to (261.9, 46.0)
- moved D28 31.3 mm to (261.9, 51.6)
- moved D11 26.6 mm to (257.2, 37.3), turned to -90 degrees
- moved R3 26.4 mm to (154.0, 90.1)
- moved R6 25.4 mm to (121.4, 90.1)
- moved R4 24.9 mm to (155.2, 90.1), turned to -90 degrees
- moved R5 23.6 mm to (156.4, 90.1)
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Connections:
- LED1 pad 1: +5V -> +3V3
- MX11 pad 1: COL3 -> Net-(D11-A)
- MX11 pad 2: Net-(D11-A) -> COL3
- MX12 pad 1: COL4 -> Net-(D12-A)
- MX12 pad 2: Net-(D12-A) -> COL4
- MX15 pad 1: COL0 -> Net-(D15-A)
- MX15 pad 2: Net-(D15-A) -> COL0
- MX17 pad 1: COL2 -> Net-(D17-A)
- MX17 pad 2: Net-(D17-A) -> COL2
- MX19 pad 1: COL4 -> Net-(D19-A)
- MX19 pad 2: Net-(D19-A) -> COL4
- MX2 pad 1: Net-(D2-A) -> COL1
- MX2 pad 2: COL1 -> Net-(D2-A)
- MX21 pad 1: COL6 -> Net-(D21-A)
- MX21 pad 2: Net-(D21-A) -> COL6
- MX22 pad 1: COL0 -> Net-(D22-A)
- MX22 pad 2: Net-(D22-A) -> COL0
- MX23 pad 1: COL1 -> Net-(D23-A)
- MX23 pad 2: Net-(D23-A) -> COL1
- MX25 pad 1: COL3 -> Net-(D25-A)
- MX25 pad 2: Net-(D25-A) -> COL3
- MX3 pad 1: COL2 -> Net-(D3-A)
- MX3 pad 2: Net-(D3-A) -> COL2
- MX30 pad 1: COL1 -> Net-(D30-A)
- MX30 pad 2: Net-(D30-A) -> COL1
- MX32 pad 1: COL3 -> Net-(D32-A)
- MX32 pad 2: Net-(D32-A) -> COL3
- MX34 pad 1: COL5 -> Net-(D34-A)
- MX34 pad 2: Net-(D34-A) -> COL5
- MX38 pad 1: COL2 -> Net-(D38-A)
- MX38 pad 2: Net-(D38-A) -> COL2
- MX40 pad 1: COL4 -> Net-(D40-A)
- MX40 pad 2: Net-(D40-A) -> COL4
- MX5 pad 1: COL4 -> Net-(D5-A)
- MX5 pad 2: Net-(D5-A) -> COL4
- MX7 pad 1: COL6 -> Net-(D7-A)
- MX7 pad 2: Net-(D7-A) -> COL6
- MX8 pad 1: COL0 -> Net-(D8-A)
- MX8 pad 2: Net-(D8-A) -> COL0
- MX9 pad 1: COL1 -> Net-(D9-A)
- MX9 pad 2: Net-(D9-A) -> COL1
- SW1 pad A: ENCB -> ENCA
- SW1 pad B: ENCA -> ENCB
- SW1 pad S1: COL6 -> Net-(D14-A)
- SW1 pad S2: Net-(D14-A) -> COL6
- U2 pad 1: D- -> unconnected-(U2-IO1-Pad1)
- U2 pad 3: unconnected-(U2-IO2-Pad3) -> D+
- U2 pad 4: unconnected-(U2-IO3-Pad4) -> D-
- U2 pad 6: D+ -> unconnected-(U2-IO4-Pad6)
- U4 pad 31: COL5 -> ROW1
- U4 pad 35: ROW1 -> ROW2
- U4 pad 36: ROW2 -> COL0
- U4 pad 37: COL4 -> COL1
- U4 pad 38: COL3 -> COL2
- U4 pad 39: COL2 -> COL3
- U4 pad 40: COL1 -> COL4
- U4 pad 41: COL0 -> COL5
Routing:
- net +5V: track 325.8 -> 4.69 mm, vias 4 -> 0
- net GND: track 104.2 -> 266.7 mm, vias 124 -> 24
- net ROW6: track 136.9 -> 263.0 mm, vias 0 -> 2
- net +3V3: track 181.9 -> 294.2 mm, vias 4 -> 7
- net ROW1: track 162.2 -> 274.5 mm, vias 6 -> 4
- net D+: track 139.2 -> 56.9 mm
- net D-: track 138.0 -> 57.9 mm
- net ROW2: track 204.2 -> 282.5 mm, vias 7 -> 4
- net ROW5: track 176.8 -> 236.9 mm
- net Net-(D11-A): track 5.43 -> 50.5 mm
- net ROW0: track 194.1 -> 238.9 mm, vias 2 -> 4
- net ROW4: track 192.0 -> 229.7 mm
- net COL0: track 366.6 -> 403.4 mm, vias 3 -> 4
- net Net-(D28-A): track 6.82 -> 42.9 mm
- net COL2: track 331.1 -> 364.1 mm, vias 3 -> 4
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Other:
- board size 274.6 x 84.1 mm -> 274.6 x 79.4 mm
