File: HS_KS-SLD_MX/HS_KS-SLD_MX.kicad_sch (KiCad schematic)
At the start: 148 parts, among them J1 USB_C_Receptacle_USB2.0, SW1 RotaryEncoder_Switch, U1 XC6206PxxxMR, U2 SRV05-4, U3 W25Q128JVS, U4 RP2040TR7, Y1 Crystal_GND24_Small

Commit message: Routed, will DRC tomorrow
Parts:
- removed C11: 100n, Capacitor_SMD:C_0402_1005Metric, symbol Device:C_Small
- J1: footprint Connector_USB:USB_C_Receptacle_HRO_TYPE-C-31-M-12 -> PCM_marbastlib-various:USB_C_Receptacle_HRO_TYPE-C-31-M-12
- MX1, MX10, MX11, MX12, MX15, MX16, MX17, MX18, MX19, MX2, MX20, MX21, MX22, MX23, MX24, MX25, MX26, MX29, MX3, MX30, MX31, MX32, MX33, MX34, MX35, MX36, MX37, MX38, MX39, MX4, MX40, MX41, MX42, MX43, MX44, MX45, MX46, MX47, MX48, MX49, MX5, MX50, MX51, MX52, MX53, MX6, MX7, MX8, MX9: footprint kiserdesigns:HS-KS-33-MX -> kiserdesigns:HS-KS-33_Soldered-MX
Connections:
- net +3V3: now also LED1.1 (VDD)
- net +5V: no longer LED1.1 (VDD)
- net COL0: now also MX15.2 (ROW), MX22.2 (ROW), MX8.2 (ROW), U4.36 (GPIO24); no longer MX15.1 (COL), MX22.1 (COL), MX8.1 (COL), U4.41 (GPIO29/ADC3)
- net COL1: now also MX2.1 (COL), MX23.2 (ROW), MX30.2 (ROW), MX9.2 (ROW), U4.37 (GPIO25); no longer MX2.2 (ROW), MX23.1 (COL), MX30.1 (COL), MX9.1 (COL), U4.40 (GPIO28/ADC2)
- net COL2: now also MX17.2 (ROW), MX3.2 (ROW), MX38.2 (ROW), U4.38 (GPIO26/ADC0); no longer MX17.1 (COL), MX3.1 (COL), MX38.1 (COL), U4.39 (GPIO27/ADC1)
- net COL3: now also MX11.2 (ROW), MX25.2 (ROW), MX32.2 (ROW), U4.39 (GPIO27/ADC1); no longer MX11.1 (COL), MX25.1 (COL), MX32.1 (COL), U4.38 (GPIO26/ADC0)
- net COL4: now also MX12.2 (ROW), MX19.2 (ROW), MX40.2 (ROW), MX5.2 (ROW), U4.40 (GPIO28/ADC2); no longer MX12.1 (COL), MX19.1 (COL), MX40.1 (COL), MX5.1 (COL), U4.37 (GPIO25)
- net COL5: now also MX34.2 (ROW), U4.41 (GPIO29/ADC3); no longer MX34.1 (COL), U4.31 (GPIO20)
- net COL6: now also MX21.2 (ROW), MX7.2 (ROW), SW1.S2; no longer MX21.1 (COL), MX7.1 (COL), SW1.S1
- net D+: now also U2.3 (IO2); no longer U2.6 (IO4)
- net D-: now also U2.4 (IO3); no longer U2.1 (IO1)
- net ENCA: now also SW1.A; no longer SW1.B
- net ENCB: now also SW1.B; no longer SW1.A
- net ROW1: now also U4.31 (GPIO20); no longer U4.35 (GPIO23)
- net ROW2: now also U4.35 (GPIO23); no longer U4.36 (GPIO24)
- net at D14.2 (A), MX14.2 (ROW): now also SW1.S1; no longer SW1.S2
- net at D8.2 (A): now also MX8.1 (COL); no longer MX8.2 (ROW)
- net at D21.2 (A): now also MX21.1 (COL); no longer MX21.2 (ROW)
- net at D22.2 (A): now also MX22.1 (COL); no longer MX22.2 (ROW)
- net at D40.2 (A): now also MX40.1 (COL); no longer MX40.2 (ROW)
- net at D38.2 (A): now also MX38.1 (COL); no longer MX38.2 (ROW)
- net at D7.2 (A): now also MX7.1 (COL); no longer MX7.2 (ROW)
- net at D12.2 (A): now also MX12.1 (COL); no longer MX12.2 (ROW)
- net at D19.2 (A): now also MX19.1 (COL); no longer MX19.2 (ROW)
- net at D3.2 (A): now also MX3.1 (COL); no longer MX3.2 (ROW)
- net at D15.2 (A): now also MX15.1 (COL); no longer MX15.2 (ROW)
- net at D9.2 (A): now also MX9.1 (COL); no longer MX9.2 (ROW)
- net at D30.2 (A): now also MX30.1 (COL); no longer MX30.2 (ROW)
- net at D32.2 (A): now also MX32.1 (COL); no longer MX32.2 (ROW)
- net at D34.2 (A): now also MX34.1 (COL); no longer MX34.2 (ROW)
- net at D23.2 (A): now also MX23.1 (COL); no longer MX23.2 (ROW)
- net at D17.2 (A): now also MX17.1 (COL); no longer MX17.2 (ROW)
- net at D11.2 (A): now also MX11.1 (COL); no longer MX11.2 (ROW)
- net at D25.2 (A): now also MX25.1 (COL); no longer MX25.2 (ROW)
- net at D2.2 (A): now also MX2.2 (ROW); no longer MX2.1 (COL)
- net at D5.2 (A): now also MX5.1 (COL); no longer MX5.2 (ROW)
Other:
- moved on the sheet: C14, C15, MX11, MX12, MX15, MX17, MX19, MX2, MX21, MX22, MX23, MX25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
